File: sao_eprom_v2/sao_eprom_v2.kicad_pcb (KiCad board)
At the start: 4 copper layers, 76 parts, among them J1 Conn_01x03, J2 USB_C_Receptacle_USB2.0, J3 sao_v2_addon_tht, Q1 RE1C002UNTCL, Q2 RE1C002ZPTL, Q3 RE1C002UNTCL, Q4 RE1C002ZPTL, Q5 RE1C002UNTCL, Q6 RE1C002ZPTL, U1 W25Q128JVS, U10 AP3012, U2 RP2040, U3 24LC00, U4 74LS573, U5 multi_eprom, U6 74LVC4245A-Q100, U7 74LS573, U8 SY8079AAC, U9 AP3012, X1 SX3M12.000M20F30TNN

Commit message: Nearly finished the design
Parts:
- removed R20: 100R, Resistor_SMD:R_0402_1005Metric_Pad0.72x0.64mm_HandSolder
- removed R21: 1K, Resistor_SMD:R_0402_1005Metric_Pad0.72x0.64mm_HandSolder
- R1: value 10K -> 100R
- R2: value 10K -> 1K
- moved R2 80.2 mm to (144.2, 49.0), turned to 90 degrees
- moved R7 76.3 mm to (141.0, 73.1), turned to 90 degrees
- moved R1 76.0 mm to (140.2, 49.0), turned to 90 degrees
- moved R6 75.5 mm to (140.0, 73.1), turned to 90 degrees
- moved J1 64.7 mm to (132.5, 32.8), turned to 90 degrees
- moved R3 64.5 mm to (129.1, 57.5)
- moved R4 64.4 mm to (129.1, 66.5)
- moved R5 64.4 mm to (129.1, 65.5)
- moved C9 43.2 mm to (160.8, 33.2)
- moved D4 43.2 mm to (158.0, 32.7)
- moved L2 43.2 mm to (155.5, 32.9)
- moved R12 43.2 mm to (154.0, 32.9)
- moved R14 43.2 mm to (154.0, 36.6)
- moved U9 43.2 mm to (157.0, 36.0)
- moved C8 43.1 mm to (160.8, 36.5)
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Connections:
- net Net-(J1-Pin_1) renamed /SWD_DATA
- net Net-(J1-Pin_3) renamed /SWD_CLK
- D1 pad 1: /EPROM and level shifters/Q15 -> /EPROM and level shifters/VppB
- D1 pad 2: Net-(D1-A) -> /EPROM and level shifters/~{OE}
- D2 pad 1: /EPROM and level shifters/VppB -> /EPROM and level shifters/Q15
- D2 pad 2: /EPROM and level shifters/~{OE} -> Net-(D2-A)
- R1 pad 1: /Power generation/5VEN -> /Power generation/VdetEN
- R1 pad 2: GND -> Net-(Q5-G)
- R2 pad 1: /Power generation/12V75EN -> /Power generation/12V75
- R2 pad 2: GND -> Net-(Q5-D)
- U10 pad 4: /Power generation/12V75EN -> +3V3
- U2 pad 34: /Power generation/5VEN -> unconnected-(U2-GPIO22-Pad34)
- U2 pad 35: /Power generation/12V75EN -> unconnected-(U2-GPIO23-Pad35)
- U7 pad 19: Net-(D1-A) -> Net-(D2-A)
- U9 pad 4: /Power generation/5VEN -> +3V3
Routing:
- net +5V: track 11.0 -> 89.2 mm, vias 1 -> 2
- net /Power generation/VppAEN: track 0.00 -> 46.9 mm, vias 0 -> 2
- net /EPROM and level shifters/AHS: track 0.00 -> 45.1 mm, vias 0 -> 3
- net /EPROM and level shifters/OE: track 0.00 -> 44.7 mm, vias 0 -> 2
- net /Power generation/VppBEN: track 0.00 -> 44.4 mm, vias 0 -> 2
- net /EPROM and level shifters/VppB: track 1.70 -> 44.5 mm, vias 0 -> 1
- net /EPROM and level shifters/Q9: track 1.70 -> 42.3 mm, vias 0 -> 1
- net /EPROM and level shifters/Q15: track 1.70 -> 40.7 mm, vias 0 -> 1
- net /Power generation/VdetEN: track 0.00 -> 36.7 mm, vias 0 -> 2
- net /EPROM and level shifters/Q10: track 0.00 -> 35.2 mm, vias 0 -> 1
- net SDA: track 0.00 -> 33.5 mm, vias 0 -> 2
- net /EPROM and level shifters/~{OE}: track 0.00 -> 32.3 mm, vias 0 -> 2
- net SCL: track 0.00 -> 32.1 mm, vias 0 -> 2
- net /EPROM and level shifters/Q11: track 0.00 -> 30.9 mm, vias 0 -> 1
- net /SWD_CLK: track 0.00 -> 30.0 mm
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- added copper zone on In2.Cu, net +3V3
- added copper zone on B.Cu, net GND
- added copper zone on F.Cu, net GND
- added copper zone on In1.Cu, net GND
Other:
- board outline added: 65.1 x 55.1 mm
- board text added: "+3V3"
- board text added: "1.5mm clearance"
- board text added: "CLK"
- board text added: "DATA"
- board text added: "DEBUG"
- board text added: "GND"
- board text added: "IO1"
- board text added: "IO2"
- board text added: "SCL"
- board text added: "SDA"
- board text added: "ZIF socket area keep out footprints"

Commit message: First complete PCB
Parts:
- added REF**: RobotMan2412_20mm, RobotMan2412:RobotMan2412_20mm, B.Cu at (139.8, 61.0)
Connections:
- U2 pad 26: ~{RST} -> +3V3
Routing:
- net +3V3: track 74.0 -> 77.4 mm, vias 17 -> 18
- net ~{RST}: track 3.37 -> 0.00 mm, vias 1 -> 0
Other:
- board text added: "12.75V"
- board text added: "3.3V"
- board text added: "5V"
- board text added: "Address high"
- board text added: "Address low"
- board text added: "EPROM"
- board text added: "Identification"
- board text added: "Level shifter"
- board text added: "Power switches"
- board text added: "Program"
