File: sao_eprom_v2/eprom.kicad_sch (KiCad schematic)
At the start: 32 parts, among them U4 74LS573, U7 74LS573

Commit message: Candidate revision No. 1
Parts:
- removed D4 (x3): 1N5819WS, Diode_SMD:D_SOD-323_HandSoldering, symbol Diode:1N5819WS
- added D1, D2, D3: 1N4007, Diode_SMD:D_SOD-323_HandSoldering, symbol Device:D
Connections:
- net Vdet: now also D3.1 (K)
- net VppA: now also D2.1 (K)
- net VppB: now also D1.1 (K)
- net ~{OE}: now also D1.2 (A)
- net at U7.13 (Q6): now also D3.2 (A)
- net at U7.19 (Q0): now also D2.2 (A)
Changed lines of the file:
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@@
+    )
+  )
+  (symbol (lib_id "Device:D") (at 87.63 116.84 180) (unit 1)
+    (in_bom yes) (on_board yes) (dnp no) (fields_autoplaced)
+    (property "Reference" "D2" (at 87.63 110.49 0)
+      (effects (font (size 1.27 1.27)))
+    )
+    (property "Value" "1N4007" (at 87.63 113.03 0)
+      (effects (font (size 1.27 1.27)))
+    )
+    (property "Footprint" "Diode_SMD:D_SOD-323_HandSoldering" (at 87.63 116.84 0)
+      (effects (font (size 1.27 1.27)) hide)
+    )
+    (property "Datasheet" "~" (at 87.63 116.84 0)
+      (effects (font (size 1.27 1.27)) hide)
+    )
+    (property "Sim.Device" "D" (at 87.63 116.84 0)
+      (effects (font (size 1.27 1.27)) hide)
+    )
+    (property "Sim.Pins" "1=K 2=A" (at 87.63 116.84 0)
+      (effects (font (size 1.27 1.27)) hide)
+    )
+    (pin "1")
+    (pin "2")
+    (instances
+      (project "sao_eprom_v2"
+        (path "/07beccdd-32b3-4f03-aa51-fb5544b6f2d4/1053addf-4f12-44cd-9743-7d35ca2d08ac"
+          (reference "D2") (unit 1)
+        )
+      )
     )
   )
@@
         (path "/07beccdd-32b3-4f03-aa51-fb5544b6f2d4/1053addf-4f12-44cd-9743-7d35ca2d08ac"
           (reference "C26") (unit 1)
+        )
+      )
+    )
+  )
+  (symbol (lib_id "Device:D") (at 87.63 101.6 180) (unit 1)
+    (in_bom yes) (on_board yes) (dnp no) (fields_autoplaced)
+    (property "Reference" "D3" (at 87.63 95.25 0)
+      (effects (font (size 1.27 1.27)))
+    )
+    (property "Value" "1N4007" (at 87.63 97.79 0)
+      (effects (font (size 1.27 1.27)))
+    )
+    (property "Footprint" "Diode_SMD:D_SOD-323_HandSoldering" (at 87.63 101.6 0)
+      (effects (font (size 1.27 1.27)) hide)
+    )
+    (property "Datasheet" "~" (at 87.63 101.6 0)
+      (effects (font (size 1.27 1.27)) hide)
+    )
+    (property "Sim.Device" "D" (at 87.63 101.6 0)
+      (effects (font (size 1.27 1.27)) hide)
+    )
+    (property "Sim.Pins" "1=K 2=A" (at 87.63 101.6 0)
+      (effects (font (size 1.27 1.27)) hide)
+    )
+    (pin "1")
+    (pin "2")
+    (instances
+      (project "sao_eprom_v2"
+        (path "/07beccdd-32b3-4f03-aa51-fb5544b6f2d4/1053addf-4f12-44cd-9743-7d35ca2d08ac"
+          (reference "D3") (unit 1)
+        )
+      )
+    )
+  )
+  (symbol (lib_id "Device:D") (at 87.63 127 180) (unit 1)
+    (in_bom yes) (on_board yes) (dnp no) (fields_autoplaced)
+    (property "Reference" "D1" (at 87.63 120.65 0)
+      (effects (font (size 1.27 1.27)))
+    )
+    (property "Value" "1N4007" (at 87.63 123.19 0)
+      (effects (font (size 1.27 1.27)))
+    )
+    (property "Footprint" "Diode_SMD:D_SOD-323_HandSoldering" (at 87.63 127 0)
+      (effects (font (size 1.27 1.27)) hide)
+    )
+    (property "Datasheet" "~" (at 87.63 127 0)
+      (effects (font (size 1.27 1.27)) hide)
+    )
+    (property "Sim.Device" "D" (at 87.63 127 0)
+      (effects (font (size 1.27 1.27)) hide)
+    )
+    (property "Sim.Pins" "1=K 2=A" (at 87.63 127 0)
+      (effects (font (size 1.27 1.27)) hide)
+    )
+    (pin "1")
+    (pin "2")
+    (instances
+      (project "sao_eprom_v2"
+        (path "/07beccdd-32b3-4f03-aa51-fb5544b6f2d4/1053addf-4f12-44cd-9743-7d35ca2d08ac"
+          (reference "D1") (unit 1)
         )
       )
@@
     )
   )
-  (symbol (lib_id "Diode:1N5819WS") (at 87.63 101.6 180) (unit 1)
-    (in_bom yes) (on_board yes) (dnp no) (fields_autoplaced)
-    (property "Reference" "D4" (at 87.9475 95.25 0)
-      (effects (font (size 1.27 1.27)))
-    )
-    (property "Value" "1N5819WS" (at 87.9475 97.79 0)
-      (effects (font (size 1.27 1.27)))
-    )
-    (property "Footprint" "Diode_SMD:D_SOD-323_HandSoldering" (at 87.63 97.155 0)
-      (effects (font (size 1.27 1.27)) hide)
-    )
-    (property "Datasheet" "https://datasheet.lcsc.com/lcsc/2204281430_Guangdong-Hottech-1N5819WS_C191023.pdf" (at 87.63 101.6 0)
-      (effects (font (size 1.27 1.27)) hide)
-    )
-    (pin "1")
-    (pin "2")
-    (instances
-      (project "sao_eprom_v2"
-        (path "/07beccdd-32b3-4f03-aa51-fb5544b6f2d4/e608ecd4-0557-4bb4-9ac0-2ae7e9dd9344"
-          (reference "D4") (unit 1)
-        )
-        (path "/07beccdd-32b3-4f03-aa51-fb5544b6f2d4/1053addf-4f12-44cd-9743-7d35ca2d08ac"
-          (reference "D3") (unit 1)
-        )
-      )
-      (project "vfd"
-        (path "/c6c7f0b1-e719-4cc4-9f66-98fb677fcafc"
-          (reference "D1") (unit 1)
-        )
-      )
-    )
-  )
   (symbol (lib_id "Connector:TestPoint") (at 54.61 149.86 270) (unit 1)
     (in_bom yes) (on_board yes) (dnp no) (fields_autoplaced)
@@
     )
   )
-  (symbol (lib_id "Diode:1N5819WS") (at 87.63 127 180) (unit 1)
-    (in_bom yes) (on_board yes) (dnp no) (fields_autoplaced)
-    (property "Reference" "D4" (at 87.9475 120.65 0)
-      (effects (font (size 1.27 1.27)))
-    )
-    (property "Value" "1N5819WS" (at 87.9475 123.19 0)
-      (effects (font (size 1.27 1.27)))
-    )
-    (property "Footprint" "Diode_SMD:D_SOD-323_HandSoldering" (at 87.63 122.555 0)
-      (effects (font (size 1.27 1.27)) hide)
-    )
-    (property "Datasheet" "https://datasheet.lcsc.com/lcsc/2204281430_Guangdong-Hottech-1N5819WS_C191023.pdf" (at 87.63 127 0)
-      (effects (font (size 1.27 1.27)) hide)
-    )
-    (pin "1")
-    (pin "2")
-    (instances
-      (project "sao_eprom_v2"
-        (path "/07beccdd-32b3-4f03-aa51-fb5544b6f2d4/e608ecd4-0557-4bb4-9ac0-2ae7e9dd9344"
-          (reference "D4") (unit 1)
-        )
-        (path "/07beccdd-32b3-4f03-aa51-fb5544b6f2d4/1053addf-4f12-44cd-9743-7d35ca2d08ac"
-          (reference "D1") (unit 1)
-        )
-      )
-      (project "vfd"
-        (path "/c6c7f0b1-e719-4cc4-9f66-98fb677fcafc"
-          (reference "D1") (unit 1)
-        )
-      )
-    )
-  )
   (symbol (lib_id "power:GND") (at 58.42 38.1 270) (mirror x) (unit 1)
     (in_bom yes) (on_board yes) (dnp no) (fields_autoplaced)
@@
         )
       )
-    )
-  )
-  (symbol (lib_id "Diode:1N5819WS") (at 87.63 116.84 180) (unit 1)
-    (in_bom yes) (on_board yes) (dnp no) (fields_autoplaced)
-    (property "Reference" "D4" (at 87.9475 110.49 0)
-      (effects (font (size 1.27 1.27)))
-    )
-    (property "Value" "1N5819WS" (at 87.9475 113.03 0)
-      (effects (font (size 1.27 1.27)))
-    )
-    (property "Footprint" "Diode_SMD:D_SOD-323_HandSoldering" (at 87.63 112.395 0)
-      (effects (font (size 1.27 1.27)) hide)
-    )
-    (property "Datasheet" "https://datasheet.lcsc.com/lcsc/2204281430_Guangdong-Hottech-1N5819WS_C191023.pdf" (at 87.63 116.84 0)
-      (effects (font (size 1.27 1.27)) hide)
-    )
-    (pin "1")
-    (pin "2")
-    (instances
-      (project "sao_eprom_v2"
-        (path "/07beccdd-32b3-4f03-aa51-fb5544b6f2d4/e608ecd4-0557-4bb4-9ac0-2ae7e9dd9344"
-          (reference "D4") (unit 1)
-        )
-        (path "/07beccdd-32b3-4f03-aa51-fb5544b6f2d4/1053addf-4f12-44cd-9743-7d35ca2d08ac"
-          (reference "D2") (unit 1)
-        )
-      )
-      (project "vfd"
-        (path "/c6c7f0b1-e719-4cc4-9f66-98fb677fcafc"
-          (reference "D1") (unit 1)
-        )
-      )
