File: sao_keyboard/sao_keyboard.kicad_pcb (KiCad board)
At the start: 2 copper layers, 96 x 25.5 mm, 3 parts

Commit message: Keyboard addon Rev. 1
Parts:
- added C1: 100n, Capacitor_SMD:C_0402_1005Metric_Pad0.74x0.62mm_HandSolder, B.Cu at (160.2, 82.1)
- added C2: 100n, Capacitor_SMD:C_0402_1005Metric_Pad0.74x0.62mm_HandSolder, B.Cu at (107.8, 86.1)
- added C3: 100n, Capacitor_SMD:C_0402_1005Metric_Pad0.74x0.62mm_HandSolder, B.Cu at (129.2, 86.1)
- added C4: 100n, Capacitor_SMD:C_0402_1005Metric_Pad0.74x0.62mm_HandSolder, B.Cu at (171.8, 86.0)
- added C5: 100n, Capacitor_SMD:C_0402_1005Metric_Pad0.74x0.62mm_HandSolder, B.Cu at (185.2, 86.1)
- added C6: 100n, Capacitor_SMD:C_0402_1005Metric_Pad0.74x0.62mm_HandSolder, B.Cu at (141.0, 86.1)
- added C7: 100n, Capacitor_SMD:C_0402_1005Metric_Pad0.74x0.62mm_HandSolder, B.Cu at (113.5, 84.0)
- added H1: MountingHole_Pad, MountingHole:MountingHole_2.2mm_M2_Pad_Via, F.Cu at (185.8, 71.2)
- added J4: I2C, qwiic:1X04_1MM_RA_GND, B.Cu at (112.5, 73.8)
- added J5: I2C, qwiic:1X04_1MM_RA_GND, B.Cu at (120.8, 73.8)
- added J6: sao_v2_addon_tht, simple_add_on_v2:sao_v2_addon_tht, F.Cu at (100.2, 73.8)
- added R1: 1K, Resistor_SMD:R_0402_1005Metric_Pad0.72x0.64mm_HandSolder, B.Cu at (93.8, 96.2)
- added R10: 1K, Resistor_SMD:R_0402_1005Metric_Pad0.72x0.64mm_HandSolder, B.Cu at (117.5, 96.2)
- added R11: 1K, Resistor_SMD:R_0402_1005Metric_Pad0.72x0.64mm_HandSolder, B.Cu at (120.0, 96.2)
- added R12: 1K, Resistor_SMD:R_0402_1005Metric_Pad0.72x0.64mm_HandSolder, B.Cu at (122.8, 96.2)
- added R13: 1K, Resistor_SMD:R_0402_1005Metric_Pad0.72x0.64mm_HandSolder, B.Cu at (125.8, 96.2)
- added R14: 1K, Resistor_SMD:R_0402_1005Metric_Pad0.72x0.64mm_HandSolder, B.Cu at (128.5, 96.2)
- added R15: 1K, Resistor_SMD:R_0402_1005Metric_Pad0.72x0.64mm_HandSolder, B.Cu at (131.0, 96.2)
- added R16: 1K, Resistor_SMD:R_0402_1005Metric_Pad0.72x0.64mm_HandSolder, B.Cu at (133.5, 96.2)
- added R17: 1K, Resistor_SMD:R_0402_1005Metric_Pad0.72x0.64mm_HandSolder, B.Cu at (136.2, 96.2)
- added R18: 1K, Resistor_SMD:R_0402_1005Metric_Pad0.72x0.64mm_HandSolder, B.Cu at (139.2, 96.2)
- added R19: 1K, Resistor_SMD:R_0402_1005Metric_Pad0.72x0.64mm_HandSolder, B.Cu at (142.0, 96.2)
- added R2: 1K, Resistor_SMD:R_0402_1005Metric_Pad0.72x0.64mm_HandSolder, B.Cu at (96.5, 96.2)
- added R20: 1K, Resistor_SMD:R_0402_1005Metric_Pad0.72x0.64mm_HandSolder, B.Cu at (144.5, 96.2)
- added R21: 1K, Resistor_SMD:R_0402_1005Metric_Pad0.72x0.64mm_HandSolder, B.Cu at (147.0, 96.2)
- added R22: 1K, Resistor_SMD:R_0402_1005Metric_Pad0.72x0.64mm_HandSolder, B.Cu at (149.5, 96.2)
- added R23: 1K, Resistor_SMD:R_0402_1005Metric_Pad0.72x0.64mm_HandSolder, B.Cu at (152.0, 96.2)
- added R24: 1K, Resistor_SMD:R_0402_1005Metric_Pad0.72x0.64mm_HandSolder, B.Cu at (154.8, 96.2)
- added R25: 1K, Resistor_SMD:R_0402_1005Metric_Pad0.72x0.64mm_HandSolder, B.Cu at (157.8, 96.2)
- added R26: 1K, Resistor_SMD:R_0402_1005Metric_Pad0.72x0.64mm_HandSolder, B.Cu at (160.5, 96.2)
- added R27: 1K, Resistor_SMD:R_0402_1005Metric_Pad0.72x0.64mm_HandSolder, B.Cu at (163.0, 96.2)
- added R28: 1K, Resistor_SMD:R_0402_1005Metric_Pad0.72x0.64mm_HandSolder, B.Cu at (165.5, 96.2)
- added R29: 1K, Resistor_SMD:R_0402_1005Metric_Pad0.72x0.64mm_HandSolder, B.Cu at (168.2, 96.2)
- added R3: 1K, Resistor_SMD:R_0402_1005Metric_Pad0.72x0.64mm_HandSolder, B.Cu at (99.0, 96.2)
- added R30: 1K, Resistor_SMD:R_0402_1005Metric_Pad0.72x0.64mm_HandSolder, B.Cu at (171.2, 96.2)
- added R31: 1K, Resistor_SMD:R_0402_1005Metric_Pad0.72x0.64mm_HandSolder, B.Cu at (174.0, 96.2)
- added R32: 1K, Resistor_SMD:R_0402_1005Metric_Pad0.72x0.64mm_HandSolder, B.Cu at (176.5, 96.2)
- added R33: 1K, Resistor_SMD:R_0402_1005Metric_Pad0.72x0.64mm_HandSolder, B.Cu at (179.0, 96.2)
- added R34: 1K, Resistor_SMD:R_0402_1005Metric_Pad0.72x0.64mm_HandSolder, B.Cu at (181.5, 96.2)
- added R35: 1K, Resistor_SMD:R_0402_1005Metric_Pad0.72x0.64mm_HandSolder, B.Cu at (184.0, 96.2)
- added R36: 1K, Resistor_SMD:R_0402_1005Metric_Pad0.72x0.64mm_HandSolder, B.Cu at (186.8, 96.2)
- added R4: 1K, Resistor_SMD:R_0402_1005Metric_Pad0.72x0.64mm_HandSolder, B.Cu at (101.5, 96.2)
- added R5: 1K, Resistor_SMD:R_0402_1005Metric_Pad0.72x0.64mm_HandSolder, B.Cu at (104.2, 96.2)
- added R6: 1K, Resistor_SMD:R_0402_1005Metric_Pad0.72x0.64mm_HandSolder, B.Cu at (107.2, 96.2)
- added R7: 1K, Resistor_SMD:R_0402_1005Metric_Pad0.72x0.64mm_HandSolder, B.Cu at (110.0, 96.2)
- added R8: 1K, Resistor_SMD:R_0402_1005Metric_Pad0.72x0.64mm_HandSolder, B.Cu at (112.5, 96.2)
- added R9: 1K, Resistor_SMD:R_0402_1005Metric_Pad0.72x0.64mm_HandSolder, B.Cu at (115.0, 96.2)
- added REF**: RobotMan2412_5mm, RobotMan2412:RobotMan2412_5mm, F.Cu at (116.2, 82.5)
- added REF**: RobotMan2412_10mm, RobotMan2412:RobotMan2412_10mm, B.Cu at (140.2, 77.0)
- added U1: 74LS245, Package_SO:TSSOP-20_4.4x6.5mm_P0.65mm, B.Cu at (102.8, 88.8)
- added U2: 74LS245, Package_SO:TSSOP-20_4.4x6.5mm_P0.65mm, B.Cu at (124.2, 88.8)
- added U3: 74LS245, Package_SO:TSSOP-20_4.4x6.5mm_P0.65mm, B.Cu at (145.8, 88.8)
- added U4: 74LS245, Package_SO:TSSOP-20_4.4x6.5mm_P0.65mm, B.Cu at (166.8, 88.8)
- added U5: 74LS245, Package_SO:TSSOP-20_4.4x6.5mm_P0.65mm, B.Cu at (180.2, 88.8)
- added U6: CH32V003F4P6, Package_SO:TSSOP-20_4.4x6.5mm_P0.65mm, B.Cu at (154.2, 80.5)
- added U7: 24LC00, Package_SO:SOIC-8_3.9x4.9mm_P1.27mm, B.Cu at (116.0, 80.5)
Connections:
- J1 pad 1: unconnected-(J1-C-Pad1) -> X0Y0
- J1 pad 10: unconnected-(J1-A-Pad10) -> X1Y1
- J1 pad 11: unconnected-(J1-A#-Pad11) -> X1Y2
- J1 pad 12: unconnected-(J1-B-Pad12) -> X1Y3
- J1 pad 2: unconnected-(J1-C#-Pad2) -> X0Y1
- J1 pad 3: unconnected-(J1-D-Pad3) -> X0Y2
- J1 pad 4: unconnected-(J1-D#-Pad4) -> X0Y3
- J1 pad 5: unconnected-(J1-E-Pad5) -> X0Y4
- J1 pad 6: unconnected-(J1-F-Pad6) -> X0Y5
- J1 pad 7: unconnected-(J1-F#-Pad7) -> X0Y6
- J1 pad 8: unconnected-(J1-G-Pad8) -> X0Y7
- J1 pad 9: unconnected-(J1-G#-Pad9) -> X1Y0
- J2 pad 1: unconnected-(J2-C-Pad1) -> X1Y4
- J2 pad 10: unconnected-(J2-A-Pad10) -> X2Y5
- J2 pad 11: unconnected-(J2-A#-Pad11) -> X2Y6
- J2 pad 12: unconnected-(J2-B-Pad12) -> X2Y7
- J2 pad 2: unconnected-(J2-C#-Pad2) -> X1Y5
- J2 pad 3: unconnected-(J2-D-Pad3) -> X1Y6
- J2 pad 4: unconnected-(J2-D#-Pad4) -> X1Y7
- J2 pad 5: unconnected-(J2-E-Pad5) -> X2Y0
- J2 pad 6: unconnected-(J2-F-Pad6) -> X2Y1
- J2 pad 7: unconnected-(J2-F#-Pad7) -> X2Y2
- J2 pad 8: unconnected-(J2-G-Pad8) -> X2Y3
- J2 pad 9: unconnected-(J2-G#-Pad9) -> X2Y4
- J3 pad 1: unconnected-(J3-C-Pad1) -> X3Y0
- J3 pad 10: unconnected-(J3-A-Pad10) -> X4Y1
- J3 pad 11: unconnected-(J3-A#-Pad11) -> X4Y2
- J3 pad 12: unconnected-(J3-B-Pad12) -> X4Y3
- J3 pad 2: unconnected-(J3-C#-Pad2) -> X3Y1
- J3 pad 3: unconnected-(J3-D-Pad3) -> X3Y2
- J3 pad 4: unconnected-(J3-D#-Pad4) -> X3Y3
- J3 pad 5: unconnected-(J3-E-Pad5) -> X3Y4
- J3 pad 6: unconnected-(J3-F-Pad6) -> X3Y5
- J3 pad 7: unconnected-(J3-F#-Pad7) -> X3Y6
- J3 pad 8: unconnected-(J3-G-Pad8) -> X3Y7
- J3 pad 9: unconnected-(J3-G#-Pad9) -> X4Y0
Routing:
- net +3V3: track 0.00 -> 304.7 mm, vias 0 -> 10
- net Y0: track 0.00 -> 125.9 mm, vias 0 -> 6
- net Y1: track 0.00 -> 117.6 mm, vias 0 -> 6
- net Y2: track 0.00 -> 115.0 mm, vias 0 -> 6
- net Y3: track 0.00 -> 111.5 mm, vias 0 -> 5
- net Y4: track 0.00 -> 105.7 mm, vias 0 -> 5
- net Y5: track 0.00 -> 99.9 mm, vias 0 -> 5
- net Y6: track 0.00 -> 94.2 mm, vias 0 -> 5
- net Y7: track 0.00 -> 85.7 mm, vias 0 -> 6
- net SDA: track 0.00 -> 74.7 mm, vias 0 -> 4
- net SCL: track 0.00 -> 68.9 mm, vias 0 -> 4
- net X0: track 0.00 -> 67.7 mm, vias 0 -> 2
- net X4: track 0.00 -> 35.7 mm
- net X1: track 0.00 -> 34.7 mm, vias 0 -> 2
- net X3: track 0.00 -> 28.2 mm
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- added copper zone on B.Cu, net GND
- added copper zone on F.Cu, net GND
Other:
- board size 96 x 25.5 mm -> 96 x 33 mm
- board text added: "3V3"
- board text added: "GND"
- board text added: "GND/stylus"
- board text added: "IO1"
- board text added: "IO2"
- board text added: "Identifier"
- board text added: "Multiplexing"
- board text added: "Musical keyboard V1 Use a metal stylus 10 June 2023"
- board text added: "Processor"
- board text added: "QWIIC"
- board text added: "SCL"
- board text added: "SDA"
- board text added: "simple add-on V2"
