File: sao_barebones/sao_barebones.kicad_pcb (KiCad board)
At the start: 2 copper layers, 36 x 36 mm, 15 parts, among them J1 sao_v2_addon_tht, J2 I2C, J3 I2C, U1 24LC00

Commit message: o
Other:
- board text added: "1"
- board text added: "Barebones SAO with some blinkenlights julian@scheffers.net 2023"
- board text added: "UP"
Changed lines of the file:
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@@
     )
   )
+  (gr_line (start 149.25 58.25) (end 150 57.5)
+    (stroke (width 0.15) (type default)) (layer "B.SilkS"))
+  (gr_line (start 150.75 58.25) (end 149.25 58.25)
+    (stroke (width 0.15) (type default)) (layer "B.SilkS"))
+  (gr_line (start 150 57.5) (end 150.75 58.25)
+    (stroke (width 0.15) (type default)) (layer "B.SilkS"))
   (gr_circle (center 150 75) (end 168 75)
     (stroke (width 0.2) (type default)) (fill none) (layer "Edge.Cuts"))
+  (gr_text "UP" (at 150 59.25) (layer "B.SilkS")
+    (effects (font (size 1 1) (thickness 0.15)) (justify mirror))
+  )
+  (gr_text "Barebones SAO with some blinkenlights\njulian@scheffers.net 2023" (at 149.75 82.5) (layer "B.SilkS")
+    (effects (font (size 1 1) (thickness 0.15)) (justify bottom mirror))
+  )
   (gr_text "WP" (at 152.05 80.75) (layer "F.SilkS")
     (effects (font (size 1 1) (thickness 0.15)) (justify left))
@@
     (effects (font (size 1 1) (thickness 0.15)) (justify right))
   )
+  (gr_text "1" (at 142.75 66.5 -135) (layer "F.Mask")
+    (effects (font (size 0.5 0.5) (thickness 0.1) bold))
+  )
+  (gr_text "1" (at 161 76 90) (layer "F.Mask")
+    (effects (font (size 0.5 0.5) (thickness 0.1) bold))
+  )
+  (gr_text "1" (at 139 74 -90) (layer "F.Mask")
+    (effects (font (size 0.5 0.5) (thickness 0.1) bold))
+  )
+  (gr_text "1" (at 149 86.5) (layer "F.Mask")
+    (effects (font (size 0.5 0.5) (thickness 0.1) bold))
+  )
+  (gr_text "1" (at 141.25 82.25 -45) (layer "F.Mask")
+    (effects (font (size 0.5 0.5) (thickness 0.1) bold))
+  )
+  (gr_text "1" (at 157.25 83.75 45) (layer "F.Mask")
+    (effects (font (size 0.5 0.5) (thickness 0.1) bold))
+  )
+  (gr_text "1" (at 158.5 67.75 135) (layer "F.Mask")
+    (effects (font (size 0.5 0.5) (thickness 0.1) bold))
+  )
+  (gr_text "1" (at 151 64 180) (layer "F.Mask")
+    (effects (font (size 0.5 0.5) (thickness 0.1) bold))
+  )
   (segment (start 152.8 82.685786) (end 152.798011 82.683797) (width 0.25) (layer "F.Cu") (net 1))
